File: kicad_6_docs/lowpass_filters/filter_board.kicad_pcb (KiCad board)
At the start: 2 copper layers, 167.6 x 101.6 mm, 180 parts, among them J1 comp_dist_board_port, J2 ext_cv_port, J3 env_board_port, J4 lfo_board_port, J5 power_entry, Q1 BCM847, Q10 BCM847, Q11 BCM847, Q12 BCM847, Q13 BCM847, Q14 BCM847, Q15 BCM847, Q16 BCM847, Q17 MMBT3906, Q18 MMBT3904, Q2 BCM847, Q3 BCM847, Q4 BCM847, Q5 BCM847, Q6 BCM847, Q7 BCM847, Q8 MMBT3906, Q9 MMBT3904, U1 TL072, U10 LM4040DBZ-5, U2 TL072, U3 SSI2164, U4 TL072, U5 TL072, U6 TL072, U7 TL072, U9 LM4040DBZ-5

Commit message: Initial filter board layout
Parts:
- removed C53, C54: 100n, Capacitor_SMD:C_0805_2012Metric
- removed R81, R82: 2k7, Resistor_SMD:R_0805_2012Metric
- removed U10, U9: LM4040DBZ-5, Package_TO_SOT_SMD:SOT-23
- C10, C11, C12, C19, C22, C23, C24, C7: value 22n -> 22n 2.5%
- R1, R10, R69, R77: value 100k -> 330k
- R11, R2: value 330k -> 680k
- R41, R64: value 47k -> 100k
- R71, R79: value 100k -> 680k
- RV1, RV3, RV4: value 10k -> 100k
- RV10, RV7: value 1k -> 10k
- RV2: value 10k_C.D. -> 100k_C.D.
- moved C29 53.9 mm to (119.9, 109.7)
- moved C30 21.6 mm to (119.9, 117.5)
- moved J5 21.6 mm to (108.0, 118.7)
- moved R48 9.25 mm to (86.2, 56.8)
- moved C8 9.23 mm to (169.2, 52.0), turned to 180 degrees
- moved C39 8.34 mm to (198.0, 66.2)
- moved C40 8.31 mm to (201.9, 66.2)
- moved C41 7.19 mm to (88.6, 36.2)
- moved C42 7.09 mm to (92.5, 36.2)
- moved R4 7.07 mm to (97.7, 34.8)
- moved R5 7.07 mm to (97.7, 29.7)
- moved R7 7.07 mm to (97.7, 32.2)
- moved C1 7.07 mm to (97.7, 27.2)
- moved R2 7.07 mm to (97.7, 39.9)
- moved R3 7.07 mm to (97.7, 37.3)
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Connections:
- C29 pad 2: Net-(C29-Pad2) -> GND
- C30 pad 1: Net-(C29-Pad2) -> GND
- C31 pad 2: Net-(C29-Pad2) -> GND
- C32 pad 1: Net-(C29-Pad2) -> GND
- C33 pad 2: Net-(C29-Pad2) -> GND
- C34 pad 1: Net-(C29-Pad2) -> GND
- C35 pad 2: Net-(C29-Pad2) -> GND
- C36 pad 1: Net-(C29-Pad2) -> GND
- C37 pad 2: Net-(C29-Pad2) -> GND
- C38 pad 1: Net-(C29-Pad2) -> GND
- C39 pad 2: Net-(C29-Pad2) -> GND
- C40 pad 1: Net-(C29-Pad2) -> GND
- C41 pad 2: Net-(C29-Pad2) -> GND
- C42 pad 1: Net-(C29-Pad2) -> GND
- C43 pad 2: Net-(C29-Pad2) -> GND
- C44 pad 1: Net-(C29-Pad2) -> GND
- Q11 pad 1: Net-(C22-Pad1) -> Net-(C22-Pad2)
- Q11 pad 3: Net-(C18-Pad1) -> Net-(C19-Pad1)
- Q11 pad 4: Net-(C22-Pad2) -> Net-(C22-Pad1)
- Q11 pad 6: Net-(C19-Pad1) -> Net-(C18-Pad1)
- Q2 pad 1: Net-(C10-Pad1) -> Net-(C10-Pad2)
- Q2 pad 3: Net-(C6-Pad1) -> Net-(C7-Pad1)
- Q2 pad 4: Net-(C10-Pad2) -> Net-(C10-Pad1)
- Q2 pad 6: Net-(C7-Pad1) -> Net-(C6-Pad1)
- R18 pad 1: +5VA -> +15V
- R69 pad 2: -5VA -> -15V
- R77 pad 2: -5VA -> -15V
- R9 pad 1: +5VA -> +15V
- RV1 pad 1: -5VA -> -15V
- RV1 pad 3: +5VA -> +15V
- RV12 pad 1: +5VA -> +15V
- RV2 pad 1: -5VA -> -15V
- RV2 pad 3: +5VA -> +15V
- RV3 pad 3: +5VA -> +15V
- RV4 pad 3: +5VA -> +15V
- RV9 pad 1: +5VA -> +15V
Routing:
- net +15V: track 0.00 -> 667.8 mm, vias 0 -> 14
- net -15V: track 0.00 -> 534.2 mm, vias 0 -> 8
- net /CV_OUT_A: track 0.00 -> 306.9 mm, vias 0 -> 4
- net /CV_OUT_B: track 0.00 -> 235.9 mm
- net /IN_A: track 0.00 -> 216.1 mm, vias 0 -> 3
- net /OUT_A: track 0.00 -> 194.4 mm, vias 0 -> 1
- net /ENV_B_IN: track 0.00 -> 181.1 mm, vias 0 -> 2
- net /EXT_CV_B_IN: track 0.00 -> 168.2 mm, vias 0 -> 2
- net /cv_generators/SEPARATION: track 0.00 -> 164.4 mm, vias 0 -> 3
- net /cv_generators/FEEDBACK_CV_OUT_A: track 0.00 -> 134.6 mm, vias 0 -> 1
- net /cv_generators/FEEDBACK_CV_OUT_B: track 0.00 -> 132.7 mm, vias 0 -> 1
- net /LFO_A_IN: track 0.00 -> 132.2 mm, vias 0 -> 2
- net /LFO_B_IN: track 0.00 -> 124.2 mm, vias 0 -> 2
- net /cv_generators/MANUAL_FREQ: track 0.00 -> 121.7 mm, vias 0 -> 3
- net /lowpass_filter_A/feedback_VCA/WET_IN: track 0.00 -> 115.2 mm, vias 0 -> 2
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- added copper zone on B.Cu, net GND
- added copper zone on F.Cu, net GND
Other:
- board text added: "MSM STEREO LPF"
- board text added: "center A"
- board text added: "center B"
- board text added: "depth A"
- board text added: "depth B"
- board text added: "rez A"
- board text added: "rez B"
- board text removed: "STEREO LPF"

Commit message: Filter board rev 0 and outputs
Parts:
- added TP1: dry_A, TestPoint:TestPoint_Keystone_5000-5004_Miniature, B.Cu at (69.8, 99.7)
- added TP10: fb_CV_B, TestPoint:TestPoint_Keystone_5000-5004_Miniature, B.Cu at (144.8, 31.1)
- added TP2: wet_A, TestPoint:TestPoint_Keystone_5000-5004_Miniature, B.Cu at (69.8, 111.1)
- added TP3: mix_A, TestPoint:TestPoint_Keystone_5000-5004_Miniature, B.Cu at (69.8, 122.6)
- added TP4: freq_CV_A, TestPoint:TestPoint_Keystone_5000-5004_Miniature, B.Cu at (74.9, 31.1)
- added TP5: fb_CV_A, TestPoint:TestPoint_Keystone_5000-5004_Miniature, B.Cu at (64.1, 31.1)
- added TP6: dry_B, TestPoint:TestPoint_Keystone_5000-5004_Miniature, B.Cu at (194.9, 99.7)
- added TP7: wet_B, TestPoint:TestPoint_Keystone_5000-5004_Miniature, B.Cu at (194.9, 111.1)
- added TP8: mix_B, TestPoint:TestPoint_Keystone_5000-5004_Miniature, B.Cu at (194.9, 122.6)
- added TP9: freq_CV_B, TestPoint:TestPoint_Keystone_5000-5004_Miniature, B.Cu at (155.6, 31.1)
Routing:
- net /lowpass_filter_B/LP_OUT: track 33.3 -> 60.8 mm, vias 0 -> 1
- net /cv_generators/FEEDBACK_CV_OUT_B: track 132.7 -> 151.0 mm, vias 1 -> 3
- net /cv_generators/FEEDBACK_CV_OUT_A: track 134.6 -> 151.3 mm, vias 1 -> 3
- net /lowpass_filter_A/LP_OUT: track 13.1 -> 29.3 mm, vias 0 -> 1
- net /IN_A: track 216.1 -> 230.1 mm, vias 3 -> 4
- net /OUT_B: track 59.5 -> 69.1 mm
- net /CV_OUT_A: track 306.9 -> 316.5 mm
- net Net-(C49-Pad2): track 25.9 -> 18.8 mm
- net -15V: track 534.2 -> 528.4 mm
- net /OUT_A: track 194.4 -> 189.6 mm
- net /IN_B: track 88.8 -> 93.4 mm
- net +15V: track 667.8 -> 663.6 mm
- net Net-(C52-Pad2): track 35.8 -> 31.6 mm
- net GND: track 60.2 -> 56.4 mm, vias 29 -> 90
- net /CV_OUT_B: track 235.9 -> 239.2 mm
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Other:
- board text added: "CV AO"
- board text added: "CV BO"
- board text added: "DRY A"
- board text added: "DRY AI"
- board text added: "DRY AO"
- board text added: "DRY B"
- board text added: "DRY BI"
- board text added: "ENV AI"
- board text added: "ENV BI"
- board text added: "EXT CV AI"
- board text added: "EXT CV BI"
- board text added: "Filter board rev 0 2022-05-24"
- board text added: "LFO AI"
- board text added: "LFO BI"
- board text added: "MIX A"
- board text added: "MIX B"
- board text added: "WET A"
- board text added: "WET AO"
- board text added: "WET B"
- board text added: "WET BO"
- board text added: "freq CV A"
- board text added: "freq CV B"
- board text added: "rez CV A"
- board text added: "rez CV B"
- board text removed: "Filter board rev 0 2022-05-22"
