File: kicad_6_docs/lowpass_filters/filter_board.kicad_sch (KiCad schematic)
At the start: 5 parts, among them J1 comp_dist_board_port, J2 ext_cv_port, J3 env_board_port, J4 lfo_board_port, J5 power_entry

Commit message: Filter board rev 0 and outputs
Parts:
- added TP1: dry_A, TestPoint:TestPoint_Keystone_5000-5004_Miniature, symbol Connector:TestPoint
- added TP10: fb_CV_B, TestPoint:TestPoint_Keystone_5000-5004_Miniature, symbol Connector:TestPoint
- added TP2: wet_A, TestPoint:TestPoint_Keystone_5000-5004_Miniature, symbol Connector:TestPoint
- added TP3: mix_A, TestPoint:TestPoint_Keystone_5000-5004_Miniature, symbol Connector:TestPoint
- added TP4: freq_CV_A, TestPoint:TestPoint_Keystone_5000-5004_Miniature, symbol Connector:TestPoint
- added TP5: fb_CV_A, TestPoint:TestPoint_Keystone_5000-5004_Miniature, symbol Connector:TestPoint
- added TP6: dry_B, TestPoint:TestPoint_Keystone_5000-5004_Miniature, symbol Connector:TestPoint
- added TP7: wet_B, TestPoint:TestPoint_Keystone_5000-5004_Miniature, symbol Connector:TestPoint
- added TP8: mix_B, TestPoint:TestPoint_Keystone_5000-5004_Miniature, symbol Connector:TestPoint
- added TP9: freq_CV_B, TestPoint:TestPoint_Keystone_5000-5004_Miniature, symbol Connector:TestPoint
Connections:
- net CV_OUT_A: now also TP4.1
- net CV_OUT_B: now also TP9.1
- net IN_A: now also TP1.1
- net IN_B: now also TP6.1
- net OUT_A: now also TP3.1
- net OUT_B: now also TP8.1
- net cv_generators/FEEDBACK_CV_OUT_A: now also TP5.1
- net cv_generators/FEEDBACK_CV_OUT_B: now also TP10.1
- net lowpass_filter_A/LP_OUT: now also TP2.1
- net lowpass_filter_B/LP_OUT: now also TP7.1
Other:
- moved on the sheet: J1, J3, J4
