File: kicad_6_docs/lowpass_filters/power_supply.kicad_sch (KiCad schematic)
At the start: 29 parts, among them U1 TL072, U10 LM4040DBZ-5, U2 TL072, U3 SSI2164, U4 TL072, U5 TL072, U6 TL072, U7 TL072, U9 LM4040DBZ-5

Commit message: Initial filter board layout
Parts:
- removed C53, C54: 100n, Capacitor_SMD:C_0805_2012Metric, symbol Device:C
- removed R81, R82: 2k7, Resistor_SMD:R_0805_2012Metric, symbol Device:R
- removed U10, U9: LM4040DBZ-5, Package_TO_SOT_SMD:SOT-23, symbol Reference_Voltage:LM4040DBZ-5
Connections:
- net GND: now also C29.2, C30.1, C31.2, C32.1, C33.2, C34.1, C35.2, C36.1, C37.2, C38.1, C39.2, C40.1, C41.2, C42.1, C43.2, C44.1

Commit message: Filter board rev 0 and outputs
Other:
- title: (none) -> M.S.M. Stereo Lowpass Filter Pedal
Changed lines of the file:
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@@
 (kicad_sch (version 20211123) (generator eeschema)
   (paper "A4")
+  (title_block
+    (title "M.S.M. Stereo Lowpass Filter Pedal")
+    (date "2022-05-24")
+    (rev "0")
+    (comment 2 "creativecommons.org/licenses/by/4.0")
+    (comment 3 "License: CC by 4.0")
+    (comment 4 "Author: Jordan Aceto")
+  )
   (junction (at 127 110.49) (diameter 0) (color 0 0 0 0)
   )
