File: kicad_6_docs/lowpass_filters/wet_dry_mixers.kicad_sch (KiCad schematic)
At the start: 4 parts, among them U1 TL072, U5 TL072

Commit message: Filter board rev 0 and outputs
Other:
- title: (none) -> M.S.M. Stereo Lowpass Filter Pedal
Changed lines of the file:
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@@
 (kicad_sch (version 20211123) (generator eeschema)
   (paper "A4")
+  (title_block
+    (title "M.S.M. Stereo Lowpass Filter Pedal")
+    (date "2022-05-24")
+    (rev "0")
+    (comment 2 "creativecommons.org/licenses/by/4.0")
+    (comment 3 "License: CC by 4.0")
+    (comment 4 "Author: Jordan Aceto")
+  )
   (junction (at 161.29 118.11) (diameter 0) (color 0 0 0 0)
   )
