File: kicad_6_docs/envelope_follower/attenuverters.kicad_sch (KiCad schematic)
At the start: 7 parts, among them U3 TL072

Commit message: Env follower rev 0 and outputs
Parts:
- renumbered R15 to R14, R14 to R15, R17 to R16, R16 to R17
Connections:
- net GND: now also RV3.1, RV4.1; no longer RV3.3, RV4.3
- net SIGNAL_IN: now also RV3.3, RV4.3; no longer RV3.1, RV4.1
Changed lines of the file:
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@@
   (title_block
     (title "M.S.M. Stereo Lowpass Filter Pedal")
-    (date "2022-05-22")
+    (date "2022-05-26")
     (rev "0")
     (comment 2 "creativecommons.org/licenses/by/4.0")
@@
     (stroke (width 0) (type default) (color 0 0 0 0))
   )
+  (wire (pts (xy 111.76 95.25) (xy 118.11 95.25))
+    (stroke (width 0) (type default) (color 0 0 0 0))
+  )
   (wire (pts (xy 165.1 115.57) (xy 167.64 115.57))
     (stroke (width 0) (type default) (color 0 0 0 0))
@@
     (stroke (width 0) (type default) (color 0 0 0 0))
   )
+  (wire (pts (xy 167.64 77.47) (xy 175.26 77.47))
+    (stroke (width 0) (type default) (color 0 0 0 0))
+  )
+  (wire (pts (xy 144.78 74.93) (xy 147.32 74.93))
+    (stroke (width 0) (type default) (color 0 0 0 0))
+  )
+  (wire (pts (xy 135.89 118.11) (xy 149.86 118.11))
+    (stroke (width 0) (type default) (color 0 0 0 0))
+  )
+  (wire (pts (xy 118.11 113.03) (xy 132.08 113.03))
+    (stroke (width 0) (type default) (color 0 0 0 0))
+  )
+  (wire (pts (xy 132.08 86.36) (xy 132.08 83.82))
+    (stroke (width 0) (type default) (color 0 0 0 0))
+  )
+  (wire (pts (xy 147.32 74.93) (xy 149.86 74.93))
+    (stroke (width 0) (type default) (color 0 0 0 0))
+  )
+  (wire (pts (xy 167.64 115.57) (xy 176.53 115.57))
+    (stroke (width 0) (type default) (color 0 0 0 0))
+  )
+  (wire (pts (xy 165.1 77.47) (xy 167.64 77.47))
+    (stroke (width 0) (type default) (color 0 0 0 0))
+  )
+  (wire (pts (xy 132.08 114.3) (xy 132.08 113.03))
+    (stroke (width 0) (type default) (color 0 0 0 0))
+  )
+  (wire (pts (xy 135.89 80.01) (xy 149.86 80.01))
+    (stroke (width 0) (type default) (color 0 0 0 0))
+  )
+  (wire (pts (xy 167.64 66.04) (xy 161.29 66.04))
+    (stroke (width 0) (type default) (color 0 0 0 0))
+  )
+  (wire (pts (xy 132.08 74.93) (xy 118.11 74.93))
+    (stroke (width 0) (type default) (color 0 0 0 0))
+  )
   (wire (pts (xy 118.11 95.25) (xy 118.11 113.03))
-    (stroke (width 0) (type default) (color 0 0 0 0))
-  )
-  (wire (pts (xy 167.64 77.47) (xy 175.26 77.47))
-    (stroke (width 0) (type default) (color 0 0 0 0))
-  )
-  (wire (pts (xy 144.78 74.93) (xy 147.32 74.93))
-    (stroke (width 0) (type default) (color 0 0 0 0))
-  )
-  (wire (pts (xy 135.89 118.11) (xy 149.86 118.11))
-    (stroke (width 0) (type default) (color 0 0 0 0))
-  )
-  (wire (pts (xy 118.11 113.03) (xy 132.08 113.03))
-    (stroke (width 0) (type default) (color 0 0 0 0))
-  )
-  (wire (pts (xy 132.08 86.36) (xy 132.08 83.82))
-    (stroke (width 0) (type default) (color 0 0 0 0))
-  )
-  (wire (pts (xy 147.32 74.93) (xy 149.86 74.93))
-    (stroke (width 0) (type default) (color 0 0 0 0))
-  )
-  (wire (pts (xy 113.03 95.25) (xy 118.11 95.25))
-    (stroke (width 0) (type default) (color 0 0 0 0))
-  )
-  (wire (pts (xy 167.64 115.57) (xy 176.53 115.57))
-    (stroke (width 0) (type default) (color 0 0 0 0))
-  )
-  (wire (pts (xy 165.1 77.47) (xy 167.64 77.47))
-    (stroke (width 0) (type default) (color 0 0 0 0))
-  )
-  (wire (pts (xy 132.08 114.3) (xy 132.08 113.03))
-    (stroke (width 0) (type default) (color 0 0 0 0))
-  )
-  (wire (pts (xy 135.89 80.01) (xy 149.86 80.01))
-    (stroke (width 0) (type default) (color 0 0 0 0))
-  )
-  (wire (pts (xy 167.64 66.04) (xy 161.29 66.04))
-    (stroke (width 0) (type default) (color 0 0 0 0))
-  )
-  (wire (pts (xy 132.08 74.93) (xy 118.11 74.93))
     (stroke (width 0) (type default) (color 0 0 0 0))
   )
@@
     (effects (font (size 1.27 1.27)) (justify left))
   )
-  (hierarchical_label "SIGNAL_IN" (shape input) (at 113.03 95.25 180)
+  (hierarchical_label "SIGNAL_IN" (shape input) (at 111.76 95.25 180)
     (effects (font (size 1.27 1.27)) (justify right))
   )
@@
   (symbol (lib_id "Device:R") (at 140.97 74.93 90) (unit 1)
     (in_bom yes) (on_board yes) (fields_autoplaced)
-    (property "Reference" "R15" (id 0) (at 140.97 68.58 90))
+    (property "Reference" "R14" (id 0) (at 140.97 68.58 90))
     (property "Value" "100k" (id 1) (at 140.97 71.12 90))
     (property "Footprint" "Resistor_SMD:R_0805_2012Metric" (id 2) (at 140.97 76.708 90)
@@
     (pin "2")
   )
-  (symbol (lib_id "Device:R_Potentiometer") (at 132.08 118.11 0) (unit 1)
+  (symbol (lib_id "Device:R_Potentiometer") (at 132.08 118.11 0) (mirror x) (unit 1)
     (in_bom yes) (on_board yes)
-    (property "Reference" "RV4" (id 0) (at 128.27 119.38 0)
-      (effects (font (size 1.27 1.27)) (justify right))
-    )
-    (property "Value" "100k C.D." (id 1) (at 130.81 116.84 0)
+    (property "Reference" "RV4" (id 0) (at 128.27 116.84 0)
+      (effects (font (size 1.27 1.27)) (justify right))
+    )
+    (property "Value" "100k C.D." (id 1) (at 130.81 119.38 0)
       (effects (font (size 1.27 1.27)) (justify right))
     )
@@
   (symbol (lib_id "Device:R") (at 140.97 113.03 90) (unit 1)
     (in_bom yes) (on_board yes) (fields_autoplaced)
-    (property "Reference" "R17" (id 0) (at 140.97 106.68 90))
+    (property "Reference" "R16" (id 0) (at 140.97 106.68 90))
     (property "Value" "100k" (id 1) (at 140.97 109.22 90))
     (property "Footprint" "Resistor_SMD:R_0805_2012Metric" (id 2) (at 140.97 114.808 90)
@@
   (symbol (lib_id "Device:R") (at 157.48 104.14 90) (unit 1)
     (in_bom yes) (on_board yes) (fields_autoplaced)
-    (property "Reference" "R16" (id 0) (at 157.48 97.79 90))
+    (property "Reference" "R17" (id 0) (at 157.48 97.79 90))
     (property "Value" "100k" (id 1) (at 157.48 100.33 90))
     (property "Footprint" "Resistor_SMD:R_0805_2012Metric" (id 2) (at 157.48 105.918 90)
@@
   (symbol (lib_id "Device:R") (at 157.48 66.04 90) (unit 1)
     (in_bom yes) (on_board yes) (fields_autoplaced)
-    (property "Reference" "R14" (id 0) (at 157.48 59.69 90))
+    (property "Reference" "R15" (id 0) (at 157.48 59.69 90))
     (property "Value" "100k" (id 1) (at 157.48 62.23 90))
     (property "Footprint" "Resistor_SMD:R_0805_2012Metric" (id 2) (at 157.48 67.818 90)
@@
     (pin "1")
   )
-  (symbol (lib_id "Device:R_Potentiometer") (at 132.08 80.01 0) (unit 1)
+  (symbol (lib_id "Device:R_Potentiometer") (at 132.08 80.01 0) (mirror x) (unit 1)
     (in_bom yes) (on_board yes)
-    (property "Reference" "RV3" (id 0) (at 128.27 81.28 0)
-      (effects (font (size 1.27 1.27)) (justify right))
-    )
-    (property "Value" "100k C.D." (id 1) (at 130.81 78.74 0)
-      (effects (font (size 1.27 1.27)) (justify right))
-    )
+    (property "Reference" "RV3" (id 0) (at 128.27 78.74 0)
+      (effects (font (size 1.27 1.27)) (justify right))
+    )
+    (property "Value" "100k C.D." (id 1) (at 130.81 81.28 0)
+      (effects (font (size 1.27 1.27)) (justify right))
+    )
