File: kicad_6_docs/envelope_follower/envelope_follower.kicad_pcb (KiCad board)
At the start: 2 copper layers, 40.6 x 190.5 mm, 45 parts, among them J1 audio_IO, J2 vcf_board_port, J3 power_entry, U1 TL072, U2 TL072, U3 TL072

Commit message: Env follower rev 0 and outputs
Parts:
- removed the TP2 at (114.9, 41.9)
- added D3: 1N4148W, Diode_SMD:D_SOD-123, B.Cu at (121.4, 32.3)
- added D5: 1N4148W, Diode_SMD:D_SOD-123, B.Cu at (121.4, 26.7)
- added D6: 1N4148W, Diode_SMD:D_SOD-123, B.Cu at (122.4, 93.0)
- added R7: 5k6, Resistor_SMD:R_0805_2012Metric, B.Cu at (121.4, 35.1)
- added TP1: dry_audio, TestPoint:TestPoint_Keystone_5000-5004_Miniature, B.Cu at (121.2, 47.5)
- added TP4: env_A, TestPoint:TestPoint_Keystone_5000-5004_Miniature, B.Cu at (137.9, 142.7)
- added TP5: env_B, TestPoint:TestPoint_Keystone_5000-5004_Miniature, B.Cu at (121.2, 142.7)
- C1: value 22n -> 470n; footprint Capacitor_SMD:C_0805_2012Metric -> Capacitor_THT:C_Rect_L7.0mm_W3.5mm_P5.00mm
- C2: value 10u -> 220n; footprint Capacitor_THT:CP_Radial_D6.3mm_P2.50mm -> Capacitor_THT:C_Rect_L7.0mm_W3.5mm_P5.00mm
- C3: value 22n -> 10u; footprint Capacitor_SMD:C_0805_2012Metric -> Capacitor_THT:CP_Radial_D6.3mm_P2.50mm
- D4: value 5V1 -> 1N4148W
- R1: renamed from R4; value 100k -> 5k6
- R10: value 680k -> 1k
- R11: value 220k -> 680k
- R12: value 3k3 -> 220k
- R13: value 100k -> 47k
- R8, R9: value 3k3 -> 10k
- TP3: value scaled_env_-5_to_+5 -> raw_env; moved to F.Cu
- moved C3 85.0 mm to (122.4, 113.5)
- moved TP2 83.5 mm to (121.4, 20.8)
- moved R11 75.1 mm to (122.4, 106.2), turned to 0 degrees
- moved R9 72.5 mm to (136.4, 103.6), turned to 180 degrees
- moved C2 72.3 mm to (140.9, 110.0)
- moved R3 71.4 mm to (137.9, 37.6), turned to 0 degrees
- moved U2 71.0 mm to (129.5, 103.1)
- moved C8 71.0 mm to (127.5, 108.5)
- moved C9 71.0 mm to (131.6, 108.5)
- moved C6 70.6 mm to (127.5, 41.1)
- moved C7 70.6 mm to (131.6, 41.1)
- moved U1 70.6 mm to (129.5, 35.8)
- moved R13 70.0 mm to (122.4, 103.6), turned to 180 degrees
- moved R4 68.9 mm to (121.3, 37.6)
- moved D1 68.8 mm to (137.9, 34.8)
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- renumbered D2 to D1, D3 to D2, D1 to D7, R15 to R14, R14 to R15, R17 to R16, R16 to R17, R1 to R18, R7 to R3, R5 to R4, R3 to R5, TP1 to TP2
Connections:
- C1 pad 1: /fwr/SIGNAL_IN -> Net-(C1-Pad1)
- C3 pad 2: /attenuverters/SIGNAL_IN -> GND
- D4 pad 2: GND -> Net-(D3-Pad1)
- R1 pad 1: Net-(C1-Pad2) -> Net-(R1-Pad1)
- R10 pad 1: -15V -> Net-(D6-Pad2)
- R11 pad 1: Net-(C3-Pad1) -> +15V
- R11 pad 2: /attenuverters/SIGNAL_IN -> Net-(R11-Pad2)
- R12 pad 1: /gain_and_offset/SIGNAL_IN -> Net-(R11-Pad2)
- R12 pad 2: Net-(D4-Pad1) -> /attenuverters/SIGNAL_IN
- R13 pad 1: Net-(D4-Pad1) -> Net-(R11-Pad2)
- R13 pad 2: Net-(C3-Pad1) -> GND
- R18 pad 2: /gain_and_offset/SIGNAL_IN -> /attenuverters/SIGNAL_IN
- R5 pad 2: /fwr/SIGNAL_OUT -> Net-(R5-Pad2)
- R8 pad 2: Net-(R8-Pad2) -> Net-(C1-Pad1)
- R9 pad 1: Net-(R9-Pad1) -> Net-(C1-Pad1)
- R9 pad 2: GND -> Net-(C2-Pad1)
- RV1 pad 1: Net-(C2-Pad1) -> /fwr/SIGNAL_IN
- RV1 pad 2: Net-(R8-Pad2) -> /fwr/SIGNAL_IN
- RV1 pad 3: Net-(R8-Pad2) -> Net-(R1-Pad1)
- RV2 pad 1: Net-(R9-Pad1) -> Net-(C3-Pad1)
- RV2 pad 2: /gain_and_offset/SIGNAL_IN -> Net-(C1-Pad2)
- RV2 pad 3: /gain_and_offset/SIGNAL_IN -> Net-(C1-Pad2)
- RV3 pad 1: /attenuverters/SIGNAL_IN -> GND
- RV3 pad 3: GND -> /attenuverters/SIGNAL_IN
- RV4 pad 1: /attenuverters/SIGNAL_IN -> GND
- RV4 pad 3: GND -> /attenuverters/SIGNAL_IN
- U1 pad 7: /fwr/SIGNAL_OUT -> Net-(R5-Pad2)
- U2 pad 1: /gain_and_offset/SIGNAL_IN -> Net-(C1-Pad2)
- U2 pad 2: Net-(R9-Pad1) -> Net-(C1-Pad2)
- U2 pad 5: GND -> Net-(C3-Pad1)
- U2 pad 6: Net-(C3-Pad1) -> Net-(R11-Pad2)
Routing:
- net /attenuverters/SIGNAL_IN: track 0.00 -> 194.5 mm, vias 0 -> 2
- net +15V: track 0.00 -> 170.9 mm, vias 0 -> 2
- net -15V: track 0.00 -> 153.2 mm
- net /fwr/SIGNAL_OUT: track 0.00 -> 127.6 mm
- net /attenuverters/ENVELOPE_OUT_B: track 0.00 -> 114.2 mm, vias 0 -> 1
- net /attenuverters/ENVELOPE_OUT_A: track 0.00 -> 101.4 mm
- net /fwr/SIGNAL_IN: track 0.00 -> 60.9 mm, vias 0 -> 1
- net Net-(RV4-Pad2): track 0.00 -> 54.9 mm
- net Net-(C3-Pad1): track 0.00 -> 54.6 mm, vias 0 -> 2
- net Net-(C1-Pad2): track 0.00 -> 46.6 mm, vias 0 -> 1
- net Net-(D2-Pad1): track 0.00 -> 33.3 mm, vias 0 -> 2
- net Net-(D1-Pad2): track 0.00 -> 27.0 mm, vias 0 -> 2
- net Net-(R1-Pad1): track 0.00 -> 23.8 mm
- net Net-(RV3-Pad2): track 0.00 -> 20.1 mm, vias 0 -> 1
- net /DRY_AUDIO_FROM_VCF_BOARD: track 0.00 -> 20.0 mm
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- added copper zone on B.Cu, net GND
- added copper zone on F.Cu, net GND
Other:
- board size 40.6 x 190.5 mm -> 30.5 x 190.5 mm
- board text added: "DRY"
- board text added: "EF A"
- board text added: "EF B"
- board text added: "Envelope Follower rev 0 2022-05-26"
- board text added: "FWR"
- board text added: "MSM Stereo LPF"
- board text added: "NRM OUT"
- board text added: "RAW EF"
- board text removed: "Envelope Follower rev 0 2022-05-22"
- board text removed: "SIG OUT"
- board text removed: "Stereo LPF"
