File: kicad_6_docs/envelope_follower/fwr.kicad_sch (KiCad schematic)
At the start: 10 parts, among them U1 TL072

Commit message: Env follower rev 0 and outputs
Parts:
- removed C1: 22n, Capacitor_SMD:C_0805_2012Metric, symbol Device:C
- added D3, D4, D5: 1N4148W, Diode_SMD:D_SOD-123, symbol Diode:1N4148W
- added R7: 5k6, Resistor_SMD:R_0805_2012Metric, symbol Device:R
- added RV1: 100k, Potentiometer_THT:Potentiometer_Alpha_RD901F-40-00D_Single_Vertical, symbol Device:R_Potentiometer
- R1: renamed from R4; value 100k -> 5k6
- renumbered D2 to D1, D3 to D2, R7 to R3, R5 to R4, R3 to R5
Connections:
- net GND: now also D5.1 (K)
- net SIGNAL_IN: now also RV1.1, RV1.2
- net SIGNAL_OUT: now also D3.2 (A), R7.2; no longer R5.2, U1.7
- net at R1.1: now also RV1.3
- new net: D4.1 (K), D5.2 (A)
- new net: D3.1 (K), D4.2 (A)
- new net: R5.2, R7.1, U1.7
Other:
- note added: "sensitivity"
- moved on the sheet: D1, D2, R1, R2, R3, R4, R5, R6, U1A, U1B
