File: kicad_6_docs/envelope_follower/gain_and_offset.kicad_sch (KiCad schematic)
At the start: 7 parts, among them U2 TL072

Commit message: Env follower rev 0 and outputs
Parts:
- removed R13: 100k, Resistor_SMD:R_0805_2012Metric, symbol Device:R
- added RV?: 100k, Potentiometer_THT:Potentiometer_Alpha_RD901F-40-00D_Single_Vertical, symbol Device:R_Potentiometer
Connections:
- net at D4.1 (K), R12.2: now also RV?.3
- net at C3.1, R10.2, R11.1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: now also RV?.1, RV?.2
Other:
- note added: "gain"
- moved on the sheet: D4, R12
Changed lines of the file:
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@@
   (junction (at 161.29 96.52) (diameter 0) (color 0 0 0 0)
   )
-  (junction (at 125.73 96.52) (diameter 0) (color 0 0 0 0)
+  (junction (at 113.03 96.52) (diameter 0) (color 0 0 0 0)
   )
   (junction (at 161.29 87.63) (diameter 0) (color 0 0 0 0)
   )
+  (junction (at 133.35 96.52) (diameter 0) (color 0 0 0 0)
+  )
   (wire (pts (xy 161.29 96.52) (xy 175.26 96.52))
     (stroke (width 0) (type default) (color 0 0 0 0))
@@
     (stroke (width 0) (type default) (color 0 0 0 0))
   )
-  (wire (pts (xy 125.73 101.6) (xy 125.73 96.52))
+  (wire (pts (xy 127 92.71) (xy 127 90.17))
+    (stroke (width 0) (type default) (color 0 0 0 0))
+  )
+  (wire (pts (xy 127 90.17) (xy 133.35 90.17))
+    (stroke (width 0) (type default) (color 0 0 0 0))
+  )
+  (wire (pts (xy 113.03 101.6) (xy 113.03 96.52))
+    (stroke (width 0) (type default) (color 0 0 0 0))
+  )
+  (wire (pts (xy 130.81 96.52) (xy 133.35 96.52))
     (stroke (width 0) (type default) (color 0 0 0 0))
   )
@@
     (stroke (width 0) (type default) (color 0 0 0 0))
   )
-  (wire (pts (xy 125.73 109.22) (xy 125.73 111.76))
-    (stroke (width 0) (type default) (color 0 0 0 0))
-  )
-  (wire (pts (xy 109.22 96.52) (xy 115.57 96.52))
+  (wire (pts (xy 113.03 109.22) (xy 113.03 111.76))
+    (stroke (width 0) (type default) (color 0 0 0 0))
+  )
+  (wire (pts (xy 133.35 96.52) (xy 140.97 96.52))
     (stroke (width 0) (type default) (color 0 0 0 0))
   )
@@
     (stroke (width 0) (type default) (color 0 0 0 0))
   )
-  (wire (pts (xy 138.43 96.52) (xy 140.97 96.52))
-    (stroke (width 0) (type default) (color 0 0 0 0))
-  )
   (wire (pts (xy 161.29 96.52) (xy 161.29 87.63))
     (stroke (width 0) (type default) (color 0 0 0 0))
@@
     (stroke (width 0) (type default) (color 0 0 0 0))
   )
-  (wire (pts (xy 125.73 96.52) (xy 123.19 96.52))
+  (wire (pts (xy 113.03 96.52) (xy 109.22 96.52))
+    (stroke (width 0) (type default) (color 0 0 0 0))
+  )
+  (wire (pts (xy 133.35 90.17) (xy 133.35 96.52))
+    (stroke (width 0) (type default) (color 0 0 0 0))
+  )
+  (wire (pts (xy 113.03 96.52) (xy 123.19 96.52))
     (stroke (width 0) (type default) (color 0 0 0 0))
   )
@@
     (stroke (width 0) (type default) (color 0 0 0 0))
   )
-  (wire (pts (xy 125.73 96.52) (xy 130.81 96.52))
-    (stroke (width 0) (type default) (color 0 0 0 0))
-  )
   (wire (pts (xy 127 76.2) (xy 130.81 76.2))
     (stroke (width 0) (type default) (color 0 0 0 0))
+  )
+  (wire (pts (xy 97.79 96.52) (xy 101.6 96.52))
+    (stroke (width 0) (type default) (color 0 0 0 0))
+  )
+  (text "gain" (at 120.65 92.71 0)
+    (effects (font (size 1.27 1.27)) (justify left bottom))
   )
   (hierarchical_label "SIGNAL_OUT" (shape output) (at 175.26 96.52 0)
     (effects (font (size 1.27 1.27)) (justify left))
   )
-  (hierarchical_label "SIGNAL_IN" (shape input) (at 109.22 96.52 180)
+  (hierarchical_label "SIGNAL_IN" (shape input) (at 97.79 96.52 180)
     (effects (font (size 1.27 1.27)) (justify right))
   )
-  (symbol (lib_id "Device:R") (at 119.38 96.52 90) (unit 1)
-    (in_bom yes) (on_board yes) (fields_autoplaced)
-    (property "Reference" "R12" (id 0) (at 119.38 90.17 90))
-    (property "Value" "3k3" (id 1) (at 119.38 92.71 90))
-    (property "Footprint" "Resistor_SMD:R_0805_2012Metric" (id 2) (at 119.38 98.298 90)
-      (effects (font (size 1.27 1.27)) hide)
-    )
-    (property "Datasheet" "~" (id 3) (at 119.38 96.52 0)
-      (effects (font (size 1.27 1.27)) hide)
-    )
-    (pin "1")
-    (pin "2")
-  )
-  (symbol (lib_id "Device:R") (at 134.62 96.52 90) (unit 1)
-    (in_bom yes) (on_board yes) (fields_autoplaced)
-    (property "Reference" "R13" (id 0) (at 134.62 90.17 90))
-    (property "Value" "100k" (id 1) (at 134.62 92.71 90))
-    (property "Footprint" "Resistor_SMD:R_0805_2012Metric" (id 2) (at 134.62 98.298 90)
-      (effects (font (size 1.27 1.27)) hide)
-    )
-    (property "Datasheet" "~" (id 3) (at 134.62 96.52 0)
-      (effects (font (size 1.27 1.27)) hide)
-    )
-    (pin "1")
-    (pin "2")
-  )
-  (symbol (lib_id "power:GND") (at 125.73 111.76 0) (unit 1)
-    (in_bom yes) (on_board yes) (fields_autoplaced)
-    (property "Reference" "#PWR015" (id 0) (at 125.73 118.11 0)
-      (effects (font (size 1.27 1.27)) hide)
-    )
-    (property "Value" "GND" (id 1) (at 125.73 116.84 0))
-    (property "Footprint" "" (id 2) (at 125.73 111.76 0)
-      (effects (font (size 1.27 1.27)) hide)
-    )
-    (property "Datasheet" "" (id 3) (at 125.73 111.76 0)
-      (effects (font (size 1.27 1.27)) hide)
-    )
-    (pin "1")
+  (symbol (lib_id "Device:R") (at 105.41 96.52 90) (unit 1)
+    (in_bom yes) (on_board yes) (fields_autoplaced)
+    (property "Reference" "R12" (id 0) (at 105.41 90.17 90))
+    (property "Value" "3k3" (id 1) (at 105.41 92.71 90))
+    (property "Footprint" "Resistor_SMD:R_0805_2012Metric" (id 2) (at 105.41 98.298 90)
+      (effects (font (size 1.27 1.27)) hide)
+    )
+    (property "Datasheet" "~" (id 3) (at 105.41 96.52 0)
+      (effects (font (size 1.27 1.27)) hide)
+    )
+    (pin "1")
+    (pin "2")
+  )
+  (symbol (lib_id "power:GND") (at 113.03 111.76 0) (unit 1)
+    (in_bom yes) (on_board yes) (fields_autoplaced)
+    (property "Reference" "#PWR015" (id 0) (at 113.03 118.11 0)
+      (effects (font (size 1.27 1.27)) hide)
+    )
+    (property "Value" "GND" (id 1) (at 113.03 116.84 0))
+    (property "Footprint" "" (id 2) (at 113.03 111.76 0)
+      (effects (font (size 1.27 1.27)) hide)
+    )
+    (property "Datasheet" "" (id 3) (at 113.03 111.76 0)
+      (effects (font (size 1.27 1.27)) hide)
+    )
+    (pin "1")
+  )
+  (symbol (lib_id "Device:R_Potentiometer") (at 127 96.52 270) (mirror x) (unit 1)
+    (in_bom yes) (on_board yes) (fields_autoplaced)
+    (property "Reference" "RV?" (id 0) (at 127 100.33 90))
+    (property "Value" "100k" (id 1) (at 127 102.87 90))
+    (property "Footprint" "Potentiometer_THT:Potentiometer_Alpha_RD901F-40-00D_Single_Vertical" (id 2) (at 127 96.52 0)
+      (effects (font (size 1.27 1.27)) hide)
+    )
+    (property "Datasheet" "~" (id 3) (at 127 96.52 0)
+      (effects (font (size 1.27 1.27)) hide)
+    )
+    (pin "1")
+    (pin "2")
+    (pin "3")
   )
   (symbol (lib_id "Device:R") (at 134.62 76.2 90) (unit 1)
@@
     (pin "1")
   )
-  (symbol (lib_id "Device:D_Zener") (at 125.73 105.41 270) (unit 1)
-    (in_bom yes) (on_board yes) (fields_autoplaced)
-    (property "Reference" "D4" (id 0) (at 128.27 104.1399 90)
+  (symbol (lib_id "Device:D_Zener") (at 113.03 105.41 270) (unit 1)
+    (in_bom yes) (on_board yes) (fields_autoplaced)
+    (property "Reference" "D4" (id 0) (at 115.57 104.1399 90)
       (effects (font (size 1.27 1.27)) (justify left))
     )
-    (property "Value" "5V1" (id 1) (at 128.27 106.6799 90)
+    (property "Value" "5V1" (id 1) (at 115.57 106.6799 90)
       (effects (font (size 1.27 1.27)) (justify left))
     )
-    (property "Footprint" "Diode_SMD:D_SOD-123" (id 2) (at 125.73 105.41 0)
-      (effects (font (size 1.27 1.27)) hide)
-    )
-    (property "Datasheet" "~" (id 3) (at 125.73 105.41 0)
-      (effects (font (size 1.27 1.27)) hide)
-    )
+    (property "Footprint" "Diode_SMD:D_SOD-123" (id 2) (at 113.03 105.41 0)
+      (effects (font (size 1.27 1.27)) hide)
+    )
+    (property "Datasheet" "~" (id 3) (at 113.03 105.41 0)
+      (effects (font (size 1.27 1.27)) hide)
+    )
