File: kicad_6_docs/compression_and_distortion/compressor.kicad_sch (KiCad schematic)
At the start: 16 parts, among them U2 NE570

Commit message: Comp dist rev 0 and outputs
Parts:
- removed C36: 1u, Capacitor_THT:C_Rect_L7.2mm_W5.5mm_P5.00mm_FKS2_FKP2_MKS2_MKP2, symbol Device:C
- removed JP2: compression_mode, Connector_PinHeader_2.54mm:PinHeader_1x03_P2.54mm_Vertical, symbol Jumper:Jumper_3_Bridged12
- removed R37: 2M2, Resistor_SMD:R_0805_2012Metric, symbol Device:R
- added R4: 3k3, Resistor_SMD:R_0805_2012Metric, symbol Device:R
- added R8: 22k, Resistor_SMD:R_0805_2012Metric, symbol Device:R
- renumbered C31 to C1, C30 to C2, C35 to C3, C37 to C4, C33 to C5, C34 to C6, C32 to C7, R38 to R3, R39 to R5, R41 to R6, R40 to R7
Connections:
- net GND: now also R8.2
- net SIGNAL_IN: now also R4.2; no longer C2.2, RV1.1
- net SIGNAL_OUT: now also C4.1; no longer RV1.2
- net at C2.1: now also RV1.2, RV1.3, U2.2
- new net: C2.2, R4.1
- new net: R8.1, RV1.1
Other:
- note added: "compression"
- note removed: "Compression mode Jumper: Connect to input for AGC @ ~2VPP Connect to output for 2:1 compression"
- moved on the sheet: C1, C2, C3, C4, C5, C6, C7, R3, R5, R6, R7, RV1A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
