File: kicad_6_docs/compression_and_distortion/compressor_distortion.kicad_pcb (KiCad board)
At the start: 2 copper layers, 52.1 x 185.4 mm, 110 parts, among them J1 dry_in, J2 vcf_board_send_receive, J3 final_out, J4 power_entry, Q1 BS170, Q2 BF245A, Q3 BS170, Q4 BF245A, SW1 bypass_switch_A, SW2 bypass_switch_B, U1 TL072, U2 NE570, U3 TL072, U4 TL072, U5 TL072

Commit message: Comp dist rev 0 and outputs
Parts:
- removed the C14 at (110.7, 56.1)
- removed the C36 at (135.6, 56.1)
- removed JP1, JP2: compression_mode, Connector_PinHeader_2.54mm:PinHeader_1x03_P2.54mm_Vertical
- removed the R37 at (142.5, 58.2)
- removed the R9 at (126.6, 100.8)
- added C37: 100n, Capacitor_SMD:C_0805_2012Metric, B.Cu at (135.3, 136.1)
- added C38: 100n, Capacitor_SMD:C_0805_2012Metric, B.Cu at (139.3, 136.1)
- added R10: 3k3, Resistor_SMD:R_0805_2012Metric, B.Cu at (104.1, 76.5)
- added R14: 22k, Resistor_SMD:R_0805_2012Metric, B.Cu at (124.6, 83.6)
- added R24: 1M, Resistor_SMD:R_0805_2012Metric, B.Cu at (126.7, 100.6)
- added R30: 100k, Resistor_SMD:R_0805_2012Metric, B.Cu at (131.4, 132.8)
- added R4: 3k3, Resistor_SMD:R_0805_2012Metric, B.Cu at (142.2, 76.5)
- added R8: 22k, Resistor_SMD:R_0805_2012Metric, B.Cu at (120.2, 83.6)
- added U6: TL072, Package_SO:SOIC-8_3.9x4.9mm_P1.27mm, B.Cu at (117.6, 173.2)
- C17: renamed from C29; value 1u -> 100n; footprint Capacitor_THT:C_Rect_L7.2mm_W5.5mm_P5.00mm_FKS2_FKP2_MKS2_MKP2 -> Capacitor_THT:C_Rect_L7.2mm_W2.5mm_P5.00mm_FKS2_FKP2_MKS2_MKP2
- C20: renamed from C7; value 1u -> 100n; footprint Capacitor_THT:C_Rect_L7.2mm_W5.5mm_P5.00mm_FKS2_FKP2_MKS2_MKP2 -> Capacitor_THT:C_Rect_L7.2mm_W2.5mm_P5.00mm_FKS2_FKP2_MKS2_MKP2
- C21: renamed from C1; value 10u B.P. -> 1u; footprint Capacitor_THT:C_Radial_D6.3mm_H5.0mm_P2.50mm -> Capacitor_THT:C_Rect_L7.2mm_W5.5mm_P5.00mm_FKS2_FKP2_MKS2_MKP2
- C22: renamed from C2; value 10u B.P. -> 1u; footprint Capacitor_THT:C_Radial_D6.3mm_H5.0mm_P2.50mm -> Capacitor_THT:C_Rect_L7.2mm_W5.5mm_P5.00mm_FKS2_FKP2_MKS2_MKP2
- C23: renamed from C3; value 10u B.P. -> 1u; footprint Capacitor_THT:C_Radial_D6.3mm_H5.0mm_P2.50mm -> Capacitor_THT:C_Rect_L7.2mm_W5.5mm_P5.00mm_FKS2_FKP2_MKS2_MKP2
- C24: renamed from C4; value 10u B.P. -> 1u; footprint Capacitor_THT:C_Radial_D6.3mm_H5.0mm_P2.50mm -> Capacitor_THT:C_Rect_L7.2mm_W5.5mm_P5.00mm_FKS2_FKP2_MKS2_MKP2
- R16: value 2M2 -> 1M
- R22: value 1M -> 100k
- moved U4 129.9 mm to (135.4, 31.5)
- moved U3 99.1 mm to (137.3, 130.6)
- moved R16 58.8 mm to (144.8, 100.6)
- moved R22 32.0 mm to (143.1, 132.8), turned to -90 degrees
- moved TP3 30.6 mm to (105.3, 133.6)
- moved R3 17.5 mm to (142.5, 59.2), turned to 0 degrees
- moved R9 17.3 mm to (104.1, 59.2)
- moved U5 16.7 mm to (114.0, 159.4)
- moved TP4 13.2 mm to (105.3, 143.6)
- moved C3 7.88 mm to (130.6, 56.1), turned to 0 degrees
- moved C10 6.10 mm to (115.7, 56.1)
- moved C35 5.59 mm to (115.6, 167.9)
- moved R45 5.59 mm to (111.3, 174.0)
- moved C36 5.59 mm to (119.6, 167.9)
- moved R44 5.34 mm to (124.2, 174.0)
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- renumbered C31 to C1, C13 to C10, C15 to C11, C11 to C12, C12 to C13, C10 to C14, C27 to C15, C28 to C16, C5 to C18, C6 to C19, C30 to C2, C38 to C25, C39 to C26, C16 to C27, C17 to C28, C18 to C29, C35 to C3, C19 to C30, C20 to C31, C21 to C32, C22 to C33, C23 to C34, C24 to C35, C25 to C36, C26 to C39, C37 to C4, C33 to C5, C34 to C6, C32 to C7, C9 to C8, C8 to C9, D2 to D1, D1 to D2, R15 to R1, R18 to R11, R20 to R12, R19 to R13, R21 to R15, R23 to R17, R24 to R18, R25 to R19, R7 to R2, R26 to R20, R27 to R21, R8 to R23, R10 to R25, R11 to R26, R12 to R27, R13 to R28, R14 to R29, R38 to R3, R30 to R31, R31 to R32, R35 to R33, R32 to R34, R33 to R35, R34 to R36, R36 to R37, R1 to R38, R2 to R39, R3 to R40, R4 to R41, R5 to R42, R6 to R43, R28 to R44, R29 to R45, R39 to R5, R41 to R6, R40 to R7, R17 to R9
Connections:
- C11 pad 1: Net-(C15-Pad1) -> /compressor_B/SIGNAL_OUT
- C15 pad 1: Net-(C27-Pad1) -> Net-(C15-Pad1)
- C17 pad 2: /distortion_A/SIGNAL_OUT -> Net-(C17-Pad2)
- C2 pad 1: Net-(C30-Pad1) -> Net-(C2-Pad1)
- C2 pad 2: /DRY_A -> Net-(C2-Pad2)
- C20 pad 2: /distortion_B/SIGNAL_OUT -> Net-(C20-Pad2)
- C21 pad 2: Net-(C1-Pad2) (its old number) -> Net-(C21-Pad2)
- C22 pad 2: Net-(C2-Pad2) -> Net-(C22-Pad2)
- C23 pad 2: Net-(C3-Pad2) (its old number) -> Net-(C23-Pad2)
- C24 pad 2: Net-(C4-Pad2) -> Net-(C24-Pad2)
- C25 pad 1: Net-(C38-Pad1) -> Net-(C25-Pad1)
- C26 pad 1: Net-(C39-Pad1) -> Net-(C26-Pad1)
- C4 pad 1: Net-(C37-Pad1) -> /compressor_A/SIGNAL_OUT
- C9 pad 1: Net-(C8-Pad1) (its old number) -> Net-(C9-Pad1)
- C9 pad 2: /DRY_B -> Net-(C9-Pad2)
- D1 pad 1: Net-(D2-Pad1) (its old number) -> Net-(D1-Pad1)
- J3 pad 1: Net-(C1-Pad2) (its old number) -> Net-(C24-Pad2)
- J3 pad 3: Net-(C2-Pad2) -> Net-(C23-Pad2)
- J3 pad 5: Net-(C3-Pad2) (its old number) -> Net-(C22-Pad2)
- J3 pad 7: Net-(C4-Pad2) -> Net-(C21-Pad2)
- Q1 pad 1: Net-(C27-Pad1) -> Net-(C15-Pad1)
- Q1 pad 2: Net-(D2-Pad1) (its old number) -> Net-(D1-Pad1)
- R15 pad 2: Net-(D2-Pad1) (its old number) -> Net-(D1-Pad1)
- R16 pad 1: Net-(C8-Pad1) (its old number) -> Net-(C15-Pad1)
- R16 pad 2: GND -> Net-(D1-Pad1)
- R17 pad 1: Net-(D2-Pad1) (its old number) -> Net-(D1-Pad1)
- R18 pad 2: Net-(C27-Pad1) -> Net-(C15-Pad1)
- R22 pad 1: Net-(C27-Pad1) -> Net-(C17-Pad2)
- R22 pad 2: Net-(D2-Pad1) (its old number) -> GND
- R31 pad 2: Net-(C38-Pad1) -> Net-(C25-Pad1)
- R32 pad 2: Net-(C38-Pad1) -> Net-(C25-Pad1)
- R33 pad 1: Net-(C38-Pad1) -> Net-(C25-Pad1)
- R34 pad 2: Net-(C39-Pad1) -> Net-(C26-Pad1)
- R35 pad 2: Net-(R33-Pad2) -> Net-(R35-Pad2)
- R36 pad 1: Net-(R33-Pad2) -> Net-(R35-Pad2)
- R37 pad 1: Net-(C39-Pad1) -> Net-(C26-Pad1)
- R38 pad 2: Net-(C1-Pad2) (its old number) -> Net-(C21-Pad2)
- R39 pad 1: Net-(C2-Pad2) -> Net-(C22-Pad2)
- R40 pad 2: Net-(C3-Pad2) (its old number) -> Net-(C23-Pad2)
- R41 pad 1: Net-(C4-Pad2) -> Net-(C24-Pad2)
- R44 pad 2: Net-(D3-Pad2) -> Net-(D4-Pad2)
- R45 pad 2: Net-(D4-Pad2) -> Net-(D3-Pad2)
- RV1 pad 1: /DRY_A -> Net-(R8-Pad1)
- RV1 pad 2: /compressor_A/SIGNAL_OUT -> Net-(C2-Pad1)
- RV1 pad 3: Net-(C37-Pad1) -> Net-(C2-Pad1)
- RV1 pad 4: /DRY_B -> Net-(R14-Pad1)
- RV1 pad 5: /compressor_B/SIGNAL_OUT -> Net-(C9-Pad1)
- RV1 pad 6: Net-(C15-Pad1) -> Net-(C9-Pad1)
- U2 pad 15: Net-(JP1-Pad2) -> Net-(C9-Pad1)
- U2 pad 2: Net-(JP2-Pad2) -> Net-(C2-Pad1)
- U3 pad 1: /WET_A -> /distortion_A/SIGNAL_OUT
- U3 pad 2: /WET_A -> /distortion_A/SIGNAL_OUT
- U3 pad 3: /output_buffer_A/SIGNAL_IN -> Net-(C17-Pad2)
- U3 pad 5: /output_buffer_B/SIGNAL_IN -> Net-(C20-Pad2)
- U3 pad 6: /WET_B -> /distortion_B/SIGNAL_OUT
- U3 pad 7: /WET_B -> /distortion_B/SIGNAL_OUT
- U4 pad 1: /sum_diff_amp/SUM_OUT -> /WET_A
- U4 pad 2: Net-(C38-Pad1) -> /WET_A
- U4 pad 3: GND -> /output_buffer_A/SIGNAL_IN
- U4 pad 5: Net-(R33-Pad2) -> /output_buffer_B/SIGNAL_IN
- U4 pad 6: Net-(C39-Pad1) -> /WET_B
- U4 pad 7: /sum_diff_amp/DIFFERENCE_OUT -> /WET_B
- U5 pad 1: Net-(D3-Pad1) -> /sum_diff_amp/SUM_OUT
- U5 pad 2: Net-(D3-Pad2) -> Net-(C25-Pad1)
- U5 pad 3: /led_drivers/CV_A_IN -> GND
- U5 pad 5: /led_drivers/CV_B_IN -> Net-(R35-Pad2)
- U5 pad 6: Net-(D4-Pad2) -> Net-(C26-Pad1)
- U5 pad 7: Net-(D4-Pad1) -> /sum_diff_amp/DIFFERENCE_OUT
Routing:
- net +15V: track 0.00 -> 303.8 mm, vias 0 -> 4
- net /WET_B: track 0.00 -> 283.6 mm, vias 0 -> 5
- net /WET_A: track 0.00 -> 254.4 mm, vias 0 -> 4
- net -15V: track 0.00 -> 244.2 mm
- net /DRY_A: track 0.00 -> 203.2 mm
- net /DRY_B: track 0.00 -> 179.4 mm, vias 0 -> 2
- net Net-(J2-Pad4): track 0.00 -> 144.6 mm, vias 0 -> 4
- net Net-(J2-Pad8): track 0.00 -> 99.9 mm, vias 0 -> 1
- net Net-(J2-Pad7): track 0.00 -> 92.2 mm
- net Net-(J2-Pad5): track 0.00 -> 88.6 mm, vias 0 -> 2
- net /distortion_B/SIGNAL_OUT: track 0.00 -> 88.3 mm, vias 0 -> 2
- net /distortion_A/SIGNAL_OUT: track 0.00 -> 88.2 mm, vias 0 -> 2
- net Net-(C21-Pad1): track 0.00 -> 82.0 mm
- net Net-(C9-Pad1): track 0.00 -> 63.1 mm
- net Net-(C18-Pad2): track 0.00 -> 54.9 mm, vias 0 -> 1
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Other:
- board text added: "CV AI"
- board text added: "CV BI"
- board text added: "MSM Stereo LPF"
- board text removed: "COMP MODE A"
- board text removed: "COMP MODE B"
- board text removed: "CV A"
- board text removed: "CV B"
- board text removed: "Stereo LPF"
