File: kicad_6_docs/compression_and_distortion/compressor_distortion.kicad_sch (KiCad schematic)
At the start: 21 parts, among them J1 dry_in, J2 vcf_board_send_receive, J3 final_out, J4 power_entry, SW1 bypass_switch_A, SW2 bypass_switch_B

Commit message: Comp dist rev 0 and outputs
Parts:
- C21: renamed from C1; value 10u B.P. -> 1u; footprint Capacitor_THT:C_Radial_D6.3mm_H5.0mm_P2.50mm -> Capacitor_THT:C_Rect_L7.2mm_W5.5mm_P5.00mm_FKS2_FKP2_MKS2_MKP2
- C22: renamed from C2; value 10u B.P. -> 1u; footprint Capacitor_THT:C_Radial_D6.3mm_H5.0mm_P2.50mm -> Capacitor_THT:C_Rect_L7.2mm_W5.5mm_P5.00mm_FKS2_FKP2_MKS2_MKP2
- C23: renamed from C3; value 10u B.P. -> 1u; footprint Capacitor_THT:C_Radial_D6.3mm_H5.0mm_P2.50mm -> Capacitor_THT:C_Rect_L7.2mm_W5.5mm_P5.00mm_FKS2_FKP2_MKS2_MKP2
- C24: renamed from C4; value 10u B.P. -> 1u; footprint Capacitor_THT:C_Radial_D6.3mm_H5.0mm_P2.50mm -> Capacitor_THT:C_Rect_L7.2mm_W5.5mm_P5.00mm_FKS2_FKP2_MKS2_MKP2
- renumbered R1 to R38, R2 to R39, R3 to R40, R4 to R41, R5 to R42, R6 to R43
Connections:
- net at C23.2, R40.2: now also J3.3 (Pin_3); no longer J3.5 (Pin_5)
- net at C21.2, R38.2: now also J3.7 (Pin_7); no longer J3.1 (Pin_1)
- net at C24.2, R41.1: now also J3.1 (Pin_1); no longer J3.7 (Pin_7)
- net at C22.2, R39.1: now also J3.5 (Pin_5); no longer J3.3 (Pin_3)
