File: kicad_6_docs/compression_and_distortion/input_buffer.kicad_sch (KiCad schematic)
At the start: 2 parts, among them U1 TL072

Commit message: Comp dist rev 0 and outputs
Parts:
- renumbered R15 to R1
Changed lines of the file:
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@@
   (title_block
     (title "M.S.M. Stereo Lowpass Filter Pedal")
-    (date "2022-05-20")
+    (date "2022-05-26")
     (rev "0")
     (comment 2 "creativecommons.org/licenses/by/4.0")
@@
   (symbol (lib_id "Device:R") (at 139.7 101.6 0) (unit 1)
     (in_bom yes) (on_board yes) (fields_autoplaced)
-    (property "Reference" "R15" (id 0) (at 142.24 100.3299 0)
+    (property "Reference" "R1" (id 0) (at 142.24 100.3299 0)
       (effects (font (size 1.27 1.27)) (justify left))
     )
