File: kicad_6_docs/compression_and_distortion/led_drivers.kicad_sch (KiCad schematic)
At the start: 5 parts, among them U5 TL072

Commit message: Comp dist rev 0 and outputs
Parts:
- renumbered R28 to R44, R29 to R45, U5 to U6
Connections:
- net CV_A_IN: now also U6.5 (+); no longer U6.3 (+)
- net CV_B_IN: now also U6.3 (+); no longer U6.5 (+)
- net at D4.1 (KA): now also U6.1; no longer U6.7
- net at R45.2, U6.6 (-): now also D3.2 (AK); no longer D4.2 (AK)
- net at D3.1 (KA): now also U6.7; no longer U6.1
- net at R44.2, U6.2 (-): now also D4.2 (AK); no longer D3.2 (AK)
Other:
- moved on the sheet: D3, D4, R44, R45, U6A, U6B
