File: kicad_6_docs/compression_and_distortion/output_buffer.kicad_sch (KiCad schematic)
At the start: 1 part, among them U3 TL072

Commit message: Comp dist rev 0 and outputs
Parts:
- renumbered U3 to U4
Changed lines of the file:
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@@
   (title_block
     (title "M.S.M. Stereo Lowpass Filter Pedal")
-    (date "2022-05-20")
+    (date "2022-05-26")
     (rev "0")
     (comment 2 "creativecommons.org/licenses/by/4.0")
@@
   (symbol (lib_id "Amplifier_Operational:TL072") (at 128.27 88.9 0) (mirror x) (unit 1)
     (in_bom yes) (on_board yes)
-    (property "Reference" "U3" (id 0) (at 129.54 93.98 0))
+    (property "Reference" "U4" (id 0) (at 129.54 93.98 0))
     (property "Value" "TL072" (id 1) (at 130.81 96.52 0))
     (property "Footprint" "Package_SO:SOIC-8_3.9x4.9mm_P1.27mm" (id 2) (at 128.27 88.9 0)
