File: kicad_6_docs/compression_and_distortion/power_pins.kicad_sch (KiCad schematic)
At the start: 16 parts, among them U1 TL072, U2 NE570, U3 TL072, U4 TL072, U5 TL072

Commit message: Comp dist rev 0 and outputs
Parts:
- added C37, C38: 100n, Capacitor_SMD:C_0805_2012Metric, symbol Device:C
- added U6: TL072, Package_SO:SOIC-8_3.9x4.9mm_P1.27mm, symbol Amplifier_Operational:TL072
- renumbered C16 to C27, C17 to C28, C18 to C29, C19 to C30, C20 to C31, C21 to C32, C22 to C33, C23 to C34, C24 to C35, C25 to C36, C26 to C39
Connections:
- net +15V: now also C37.1, U6.8 (V+)
- net -15V: now also C38.2, U6.4 (V-)
- net GND: now also C37.2, C38.1
Changed lines of the file:
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@@
   (title_block
     (title "M.S.M. Stereo Lowpass Filter Pedal")
-    (date "2022-05-20")
+    (date "2022-05-26")
     (rev "0")
     (comment 2 "creativecommons.org/licenses/by/4.0")
@@
   (junction (at 151.13 123.19) (diameter 0) (color 0 0 0 0)
   )
+  (junction (at 179.07 123.19) (diameter 0) (color 0 0 0 0)
+  )
   (junction (at 123.19 138.43) (diameter 0) (color 0 0 0 0)
   )
+  (junction (at 165.1 138.43) (diameter 0) (color 0 0 0 0)
+  )
   (junction (at 137.16 80.01) (diameter 0) (color 0 0 0 0)
   )
@@
   (junction (at 137.16 123.19) (diameter 0) (color 0 0 0 0)
   )
+  (junction (at 165.1 59.69) (diameter 0) (color 0 0 0 0)
+  )
+  (junction (at 165.1 80.01) (diameter 0) (color 0 0 0 0)
+  )
   (junction (at 123.19 80.01) (diameter 0) (color 0 0 0 0)
   )
@@
   (junction (at 123.19 59.69) (diameter 0) (color 0 0 0 0)
   )
+  (junction (at 165.1 107.95) (diameter 0) (color 0 0 0 0)
+  )
   (junction (at 151.13 59.69) (diameter 0) (color 0 0 0 0)
   )
+  (wire (pts (xy 165.1 80.01) (xy 179.07 80.01))
+    (stroke (width 0) (type default) (color 0 0 0 0))
+  )
   (wire (pts (xy 137.16 138.43) (xy 151.13 138.43))
     (stroke (width 0) (type default) (color 0 0 0 0))
@@
     (stroke (width 0) (type default) (color 0 0 0 0))
   )
+  (wire (pts (xy 165.1 107.95) (xy 179.07 107.95))
+    (stroke (width 0) (type default) (color 0 0 0 0))
+  )
   (wire (pts (xy 137.16 80.01) (xy 151.13 80.01))
     (stroke (width 0) (type default) (color 0 0 0 0))
@@
     (stroke (width 0) (type default) (color 0 0 0 0))
   )
+  (wire (pts (xy 179.07 59.69) (xy 179.07 62.23))
+    (stroke (width 0) (type default) (color 0 0 0 0))
+  )
   (wire (pts (xy 137.16 80.01) (xy 137.16 77.47))
     (stroke (width 0) (type default) (color 0 0 0 0))
@@
     (stroke (width 0) (type default) (color 0 0 0 0))
   )
+  (wire (pts (xy 179.07 123.19) (xy 179.07 128.27))
+    (stroke (width 0) (type default) (color 0 0 0 0))
+  )
   (wire (pts (xy 151.13 107.95) (xy 151.13 110.49))
     (stroke (width 0) (type default) (color 0 0 0 0))
@@
     (stroke (width 0) (type default) (color 0 0 0 0))
   )
+  (wire (pts (xy 179.07 107.95) (xy 179.07 110.49))
+    (stroke (width 0) (type default) (color 0 0 0 0))
+  )
   (wire (pts (xy 151.13 135.89) (xy 151.13 138.43))
     (stroke (width 0) (type default) (color 0 0 0 0))
@@
     (stroke (width 0) (type default) (color 0 0 0 0))
   )
+  (wire (pts (xy 165.1 59.69) (xy 179.07 59.69))
+    (stroke (width 0) (type default) (color 0 0 0 0))
+  )
   (wire (pts (xy 137.16 110.49) (xy 137.16 107.95))
     (stroke (width 0) (type default) (color 0 0 0 0))
   )
+  (wire (pts (xy 179.07 77.47) (xy 179.07 80.01))
+    (stroke (width 0) (type default) (color 0 0 0 0))
+  )
   (wire (pts (xy 151.13 123.19) (xy 165.1 123.19))
     (stroke (width 0) (type default) (color 0 0 0 0))
   )
+  (wire (pts (xy 165.1 123.19) (xy 179.07 123.19))
+    (stroke (width 0) (type default) (color 0 0 0 0))
+  )
   (wire (pts (xy 137.16 123.19) (xy 123.19 123.19))
     (stroke (width 0) (type default) (color 0 0 0 0))
@@
     (stroke (width 0) (type default) (color 0 0 0 0))
   )
+  (wire (pts (xy 179.07 118.11) (xy 179.07 123.19))
+    (stroke (width 0) (type default) (color 0 0 0 0))
+  )
   (wire (pts (xy 165.1 77.47) (xy 165.1 80.01))
     (stroke (width 0) (type default) (color 0 0 0 0))
@@
     (stroke (width 0) (type default) (color 0 0 0 0))
   )
+  (wire (pts (xy 179.07 135.89) (xy 179.07 138.43))
+    (stroke (width 0) (type default) (color 0 0 0 0))
+  )
   (wire (pts (xy 151.13 59.69) (xy 151.13 62.23))
     (stroke (width 0) (type default) (color 0 0 0 0))
@@
     (stroke (width 0) (type default) (color 0 0 0 0))
   )
+  (wire (pts (xy 165.1 138.43) (xy 179.07 138.43))
+    (stroke (width 0) (type default) (color 0 0 0 0))
+  )
   (wire (pts (xy 123.19 107.95) (xy 123.19 110.49))
     (stroke (width 0) (type default) (color 0 0 0 0))
+  )
+  (symbol (lib_id "Amplifier_Operational:TL072") (at 181.61 69.85 0) (unit 3)
+    (in_bom yes) (on_board yes) (fields_autoplaced)
+    (property "Reference" "U6" (id 0) (at 180.34 68.5799 0)
+      (effects (font (size 1.27 1.27)) (justify left))
+    )
+    (property "Value" "TL072" (id 1) (at 180.34 71.1199 0)
+      (effects (font (size 1.27 1.27)) (justify left))
+    )
+    (property "Footprint" "Package_SO:SOIC-8_3.9x4.9mm_P1.27mm" (id 2) (at 181.61 69.85 0)
+      (effects (font (size 1.27 1.27)) hide)
+    )
+    (property "Datasheet" "http://www.ti.com/lit/ds/symlink/tl071.pdf" (id 3) (at 181.61 69.85 0)
+      (effects (font (size 1.27 1.27)) hide)
+    )
+    (pin "1")
+    (pin "2")
+    (pin "3")
+    (pin "5")
+    (pin "6")
+    (pin "7")
+    (pin "4")
+    (pin "8")
   )
   (symbol (lib_id "custom_symbols:NE570") (at 193.04 69.85 0) (mirror y) (unit 7)
@@
   (symbol (lib_id "Device:C") (at 123.19 132.08 0) (unit 1)
     (in_bom yes) (on_board yes) (fields_autoplaced)
-    (property "Reference" "C19" (id 0) (at 127 130.8099 0)
+    (property "Reference" "C30" (id 0) (at 127 130.8099 0)
       (effects (font (size 1.27 1.27)) (justify left))
     )
@@
   (symbol (lib_id "Device:C") (at 137.16 114.3 0) (unit 1)
     (in_bom yes) (on_board yes) (fields_autoplaced)
-    (property "Reference" "C20" (id 0) (at 140.97 113.0299 0)
+    (property "Reference" "C31" (id 0) (at 140.97 113.0299 0)
       (effects (font (size 1.27 1.27)) (justify left))
     )
@@
   (symbol (lib_id "Device:C") (at 151.13 132.08 0) (unit 1)
     (in_bom yes) (on_board yes) (fields_autoplaced)
-    (property "Reference" "C23" (id 0) (at 154.94 130.8099 0)
+    (property "Reference" "C34" (id 0) (at 154.94 130.8099 0)
       (effects (font (size 1.27 1.27)) (justify left))
     )
@@
   (symbol (lib_id "Device:C") (at 193.04 114.3 0) (unit 1)
     (in_bom yes) (on_board yes) (fields_autoplaced)
-    (property "Reference" "C26" (id 0) (at 196.85 113.0299 0)
+    (property "Reference" "C39" (id 0) (at 196.85 113.0299 0)
       (effects (font (size 1.27 1.27)) (justify left))
     )
@@
   (symbol (lib_id "Device:C") (at 137.16 132.08 0) (unit 1)
     (in_bom yes) (on_board yes) (fields_autoplaced)
-    (property "Reference" "C21" (id 0) (at 140.97 130.8099 0)
+    (property "Reference" "C32" (id 0) (at 140.97 130.8099 0)
       (effects (font (size 1.27 1.27)) (justify left))
     )
@@
     (pin "8")
   )
+  (symbol (lib_id "Device:C") (at 179.07 132.08 0) (unit 1)
+    (in_bom yes) (on_board yes) (fields_autoplaced)
+    (property "Reference" "C38" (id 0) (at 182.88 130.8099 0)
+      (effects (font (size 1.27 1.27)) (justify left))
+    )
+    (property "Value" "100n" (id 1) (at 182.88 133.3499 0)
+      (effects (font (size 1.27 1.27)) (justify left))
+    )
+    (property "Footprint" "Capacitor_SMD:C_0805_2012Metric" (id 2) (at 180.0352 135.89 0)
+      (effects (font (size 1.27 1.27)) hide)
+    )
+    (property "Datasheet" "~" (id 3) (at 179.07 132.08 0)
+      (effects (font (size 1.27 1.27)) hide)
+    )
+    (pin "1")
+    (pin "2")
+  )
   (symbol (lib_id "Device:C") (at 165.1 114.3 0) (unit 1)
     (in_bom yes) (on_board yes) (fields_autoplaced)
-    (property "Reference" "C24" (id 0) (at 168.91 113.0299 0)
+    (property "Reference" "C35" (id 0) (at 168.91 113.0299 0)
       (effects (font (size 1.27 1.27)) (justify left))
     )
@@
   (symbol (lib_id "Device:C") (at 151.13 114.3 0) (unit 1)
     (in_bom yes) (on_board yes) (fields_autoplaced)
-    (property "Reference" "C22" (id 0) (at 154.94 113.0299 0)
+    (property "Reference" "C33" (id 0) (at 154.94 113.0299 0)
       (effects (font (size 1.27 1.27)) (justify left))
     )
@@
   (symbol (lib_id "Device:C_Polarized") (at 99.06 132.08 0) (unit 1)
     (in_bom yes) (on_board yes) (fields_autoplaced)
-    (property "Reference" "C17" (id 0) (at 102.87 129.9209 0)
+    (property "Reference" "C28" (id 0) (at 102.87 129.9209 0)
       (effects (font (size 1.27 1.27)) (justify left))
     )
@@
   (symbol (lib_id "Device:C") (at 165.1 132.08 0) (unit 1)
     (in_bom yes) (on_board yes) (fields_autoplaced)
-    (property "Reference" "C25" (id 0) (at 168.91 130.8099 0)
+    (property "Reference" "C36" (id 0) (at 168.91 130.8099 0)
       (effects (font (size 1.27 1.27)) (justify left))
     )
@@
     (pin "1")
   )
+  (symbol (lib_id "Device:C") (at 179.07 114.3 0) (unit 1)
+    (in_bom yes) (on_board yes) (fields_autoplaced)
+    (property "Reference" "C37" (id 0) (at 182.88 113.0299 0)
+      (effects (font (size 1.27 1.27)) (justify left))
+    )
+    (property "Value" "100n" (id 1) (at 182.88 115.5699 0)
+      (effects (font (size 1.27 1.27)) (justify left))
+    )
+    (property "Footprint" "Capacitor_SMD:C_0805_2012Metric" (id 2) (at 180.0352 118.11 0)
+      (effects (font (size 1.27 1.27)) hide)
+    )
+    (property "Datasheet" "~" (id 3) (at 179.07 114.3 0)
+      (effects (font (size 1.27 1.27)) hide)
+    )
+    (pin "1")
+    (pin "2")
+  )
   (symbol (lib_id "power:-15V") (at 123.19 140.97 180) (unit 1)
     (in_bom yes) (on_board yes) (fields_autoplaced)
@@
   (symbol (lib_id "Device:C_Polarized") (at 99.06 114.3 0) (unit 1)
     (in_bom yes) (on_board yes) (fields_autoplaced)
-    (property "Reference" "C16" (id 0) (at 102.87 112.1409 0)
+    (property "Reference" "C27" (id 0) (at 102.87 112.1409 0)
       (effects (font (size 1.27 1.27)) (justify left))
     )
@@
   (symbol (lib_id "Device:C") (at 123.19 114.3 0) (unit 1)
     (in_bom yes) (on_board yes) (fields_autoplaced)
-    (property "Reference" "C18" (id 0) (at 127 113.0299 0)
-      (effects (font (size 1.27 1.27)) (justify left))
-    )
+    (property "Reference" "C29" (id 0) (at 127 113.0299 0)
+      (effects (font (size 1.27 1.27)) (justify left))
+    )
