File: kicad_6_docs/compression_and_distortion/sum_diff_amp.kicad_sch (KiCad schematic)
At the start: 10 parts, among them U4 TL072

Commit message: Comp dist rev 0 and outputs
Parts:
- renumbered C38 to C25, C39 to C26, R30 to R31, R31 to R32, R35 to R33, R32 to R34, R33 to R35, R34 to R36, R36 to R37, U4 to U5
Changed lines of the file:
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@@
   (title_block
     (title "M.S.M. Stereo Lowpass Filter Pedal")
-    (date "2022-05-20")
+    (date "2022-05-26")
     (rev "0")
     (comment 2 "creativecommons.org/licenses/by/4.0")
@@
   (symbol (lib_id "Device:R") (at 135.89 143.51 0) (unit 1)
     (in_bom yes) (on_board yes) (fields_autoplaced)
-    (property "Reference" "R34" (id 0) (at 138.43 142.2399 0)
+    (property "Reference" "R36" (id 0) (at 138.43 142.2399 0)
       (effects (font (size 1.27 1.27)) (justify left))
     )
@@
   (symbol (lib_id "Device:R") (at 146.05 64.77 90) (unit 1)
     (in_bom yes) (on_board yes) (fields_autoplaced)
-    (property "Reference" "R35" (id 0) (at 146.05 58.42 90))
+    (property "Reference" "R33" (id 0) (at 146.05 58.42 90))
     (property "Value" "100k" (id 1) (at 146.05 60.96 90))
     (property "Footprint" "Resistor_SMD:R_0805_2012Metric" (id 2) (at 146.05 66.548 90)
@@
   (symbol (lib_id "Device:R") (at 129.54 74.93 90) (unit 1)
     (in_bom yes) (on_board yes) (fields_autoplaced)
-    (property "Reference" "R31" (id 0) (at 129.54 68.58 90))
+    (property "Reference" "R32" (id 0) (at 129.54 68.58 90))
     (property "Value" "100k" (id 1) (at 129.54 71.12 90))
     (property "Footprint" "Resistor_SMD:R_0805_2012Metric" (id 2) (at 129.54 76.708 90)
@@
   (symbol (lib_id "Device:R") (at 129.54 121.92 90) (unit 1)
     (in_bom yes) (on_board yes) (fields_autoplaced)
-    (property "Reference" "R32" (id 0) (at 129.54 115.57 90))
+    (property "Reference" "R34" (id 0) (at 129.54 115.57 90))
     (property "Value" "100k" (id 1) (at 129.54 118.11 90))
     (property "Footprint" "Resistor_SMD:R_0805_2012Metric" (id 2) (at 129.54 123.698 90)
@@
   (symbol (lib_id "Device:R") (at 129.54 64.77 90) (unit 1)
     (in_bom yes) (on_board yes) (fields_autoplaced)
-    (property "Reference" "R30" (id 0) (at 129.54 58.42 90))
+    (property "Reference" "R31" (id 0) (at 129.54 58.42 90))
     (property "Value" "100k" (id 1) (at 129.54 60.96 90))
     (property "Footprint" "Resistor_SMD:R_0805_2012Metric" (id 2) (at 129.54 66.548 90)
@@
   (symbol (lib_id "Amplifier_Operational:TL072") (at 146.05 134.62 0) (mirror x) (unit 2)
     (in_bom yes) (on_board yes)
-    (property "Reference" "U4" (id 0) (at 148.59 139.7 0))
+    (property "Reference" "U5" (id 0) (at 148.59 139.7 0))
     (property "Value" "TL072" (id 1) (at 149.86 142.24 0))
     (property "Footprint" "Package_SO:SOIC-8_3.9x4.9mm_P1.27mm" (id 2) (at 146.05 134.62 0)
@@
   (symbol (lib_id "Device:R") (at 129.54 137.16 90) (unit 1)
     (in_bom yes) (on_board yes) (fields_autoplaced)
-    (property "Reference" "R33" (id 0) (at 129.54 130.81 90))
+    (property "Reference" "R35" (id 0) (at 129.54 130.81 90))
     (property "Value" "100k" (id 1) (at 129.54 133.35 90))
     (property "Footprint" "Resistor_SMD:R_0805_2012Metric" (id 2) (at 129.54 138.938 90)
@@
   (symbol (lib_id "Device:C") (at 146.05 109.22 90) (unit 1)
     (in_bom yes) (on_board yes) (fields_autoplaced)
-    (property "Reference" "C39" (id 0) (at 146.05 101.6 90))
+    (property "Reference" "C26" (id 0) (at 146.05 101.6 90))
     (property "Value" "100p" (id 1) (at 146.05 104.14 90))
     (property "Footprint" "Capacitor_SMD:C_0805_2012Metric" (id 2) (at 149.86 108.2548 0)
@@
   (symbol (lib_id "Device:C") (at 146.05 52.07 90) (unit 1)
     (in_bom yes) (on_board yes) (fields_autoplaced)
-    (property "Reference" "C38" (id 0) (at 146.05 44.45 90))
+    (property "Reference" "C25" (id 0) (at 146.05 44.45 90))
     (property "Value" "100p" (id 1) (at 146.05 46.99 90))
     (property "Footprint" "Capacitor_SMD:C_0805_2012Metric" (id 2) (at 149.86 51.1048 0)
@@
   (symbol (lib_id "Device:R") (at 146.05 121.92 90) (unit 1)
     (in_bom yes) (on_board yes) (fields_autoplaced)
-    (property "Reference" "R36" (id 0) (at 146.05 115.57 90))
+    (property "Reference" "R37" (id 0) (at 146.05 115.57 90))
     (property "Value" "100k" (id 1) (at 146.05 118.11 90))
     (property "Footprint" "Resistor_SMD:R_0805_2012Metric" (id 2) (at 146.05 123.698 90)
@@
   (symbol (lib_id "Amplifier_Operational:TL072") (at 146.05 77.47 0) (mirror x) (unit 1)
     (in_bom yes) (on_board yes)
-    (property "Reference" "U4" (id 0) (at 148.59 82.55 0))
+    (property "Reference" "U5" (id 0) (at 148.59 82.55 0))
     (property "Value" "TL072" (id 1) (at 149.86 85.09 0))
     (property "Footprint" "Package_SO:SOIC-8_3.9x4.9mm_P1.27mm" (id 2) (at 146.05 77.47 0)
