File: circuit_boards/LFO_and_PS/kicad_6/power_supply.kicad_sch (KiCad schematic)
At the start: 41 parts, among them U1 TL072, U4 LM317_TO-220, U5 L78L33_SOT89, U6 LM337_TO220

Commit message: Update PCB files, fix VCF mix polarity
Parts:
- C10, C14: footprint Capacitor_THT:CP_Radial_D17.0mm_P7.50mm -> Capacitor_THT:CP_Radial_D18.0mm_P7.50mm
Changed lines of the file:
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@@
       (effects (font (size 1.27 1.27)) (justify left))
     )
-    (property "Footprint" "Capacitor_THT:CP_Radial_D17.0mm_P7.50mm" (id 2) (at 80.9752 87.63 0)
+    (property "Footprint" "Capacitor_THT:CP_Radial_D18.0mm_P7.50mm" (id 2) (at 80.9752 87.63 0)
       (effects (font (size 1.27 1.27)) hide)
     )
@@
       (effects (font (size 1.27 1.27)) (justify left))
     )
-    (property "Footprint" "Capacitor_THT:CP_Radial_D17.0mm_P7.50mm" (id 2) (at 80.9752 71.12 0)
-      (effects (font (size 1.27 1.27)) hide)
-    )
+    (property "Footprint" "Capacitor_THT:CP_Radial_D18.0mm_P7.50mm" (id 2) (at 80.9752 71.12 0)
+      (effects (font (size 1.27 1.27)) hide)
+    )
